Commit message: Added services

File: urdf/group7bot.xacro (robot description, xacro)
@@ -1,4 +1,4 @@
 <?xml version="1.0" ?>
-    <robot name="week7bot">
+    <robot name="group7bot">
     <!-- Create a robot chassis as Base Link -->
     <link name="base_link">
@@ -154,90 +154,3 @@
          <child link="laser_sensor"/>
     </joint>
-    <!--specifying color in Gazebo-->
-    <gazebo reference="base_link">
-        <material>Gazebo/Blue</material>
-    </gazebo>
-    <gazebo reference="left_wheel">
-        <material>Gazebo/Red</material>
-    </gazebo>
-    <gazebo reference="right_wheel">
-        <material>Gazebo/Red</material>
-    </gazebo>
-    <gazebo reference="camera_link">
-        <material>Gazebo/Yellow</material>
-        <sensor name="camera" type="camera">
-            <pose> 0 0 0 0 0 0 </pose>
-            <visualize>true</visualize>
-            <update_rate>10</update_rate>
-            <camera>
-                <horizontal_fov>1.089</horizontal_fov>
-                <image>
-                    <format>R8G8B8</format>
-                    <width>640</width>
-                    <height>480</height>
-                </image>
-                <clip>
-                    <near>0.05</near>
-                    <far>8.0</far>
-                </clip>
-            </camera>
-            <plugin name="camera_controller" filename="libgazebo_ros_camera.so">
-                <frame_name>camera_link_optical</frame_name>
-                <imageTopicName>image_raw</imageTopicName>
-                <always_on>1</always_on>
-                <update_rate>30</update_rate>
-            </plugin>
-        </sensor>
-    </gazebo>
-    <!--To add the sensor behaviour, we use the laser gazebo plugin-->
-    <gazebo reference="laser_sensor">
-        <sensor type="ray" name="head_hokuyo_sensor">
-            <pose>0 0 0 0 0 0</pose>
-            <visualize>true</visualize>
-            <update_rate>20</update_rate>
-            <ray>
-                <scan>
-                    <horizontal>
-                        <samples>720</samples>
-                        <resolution>1</resolution>
-                        <min_angle>-1.570796</min_angle>
-                        <max_angle>1.570796</max_angle>
-                    </horizontal>
-                </scan>
-                <range>
-                    <min>0.10</min>
-                    <max>10.0</max>
-                    <resolution>0.01</resolution>
-                </range>
-                <noise>
-                    <type>gaussian</type>
-                    <mean>0.0</mean>
-                    <stddev>0.01</stddev>
-                </noise>
-            </ray>
-            <plugin name="gazebo_ros_head_hokuyo_controller" filename="libgazebo_ros_laser.so">
-                <topicName>/week7bot/laser/scan</topicName>
-                <frameName>laser_sensor</frameName>
-            </plugin>
-        </sensor>
-    </gazebo>
-    <gazebo>
-        <plugin filename="libgazebo_ros_diff_drive.so" name="differential_drive_controller">
-            <alwaysOn>true</alwaysOn>
-            <updateRate>20</updateRate>
-            <leftJoint>joint_left_wheel</leftJoint>
-            <rightJoint>joint_right_wheel</rightJoint>
-            <wheelSeparation>0.4</wheelSeparation>
-            <wheelDiameter>0.2</wheelDiameter>
-            <torque>0.1</torque>
-            <commandTopic>week7bot/cmd_vel</commandTopic>
-            <odometryTopic>odom</odometryTopic>
-            <odometryFrame>odom</odometryFrame>
-            <robotBaseFrame>base_link</robotBaseFrame>
-            <publishWheelTF>true</publishWheelTF>
-            <publishOdom>true</publishOdom>
-            <publishWheelJointState>true</publishWheelJointState>
-            <legacyMode>true</legacyMode>
-        </plugin>
-    </gazebo>
 </robot>
